File: main_board/Doppelganger.sch (KiCad schematic (older format))
At the start: 68 parts, among them J1 RJ45, J2 BROOK_FB, P1 BORNIER_10, P2 BORNIER_10, P3 CONN_01X06, P4 CONN_01X06, P5 TTL Serial, P6 Status Leds, SW1 SW_PUSH, SW2 SW_PUSH, U1 74HC32, U2 SIP32510, U4 74LVC07, U5 74LVC07, U6 74LVC07, U8 18F45K50, U9 MAX4737

Commit message: Pre teardrops
Parts:
- added J3: dnf, Doppelganger:GS2, symbol GS2
- added S1: dnf, Doppelganger:Sakura_solder_mask, symbol Sakura
- C1, C10, C2, C3, C4, C5, C6, C8, C9: Descr (none) -> Capacitor X7R 0.1µF 50V 10%; Farnell CC 2496944 -> 1759037; Manufacturer (none) -> MULTICOMP; Part number (none) -> MC0603B104K250CT
- C11: Descr (none) -> Capacitor X7R 4.7µF 50V 10% 0603; Farnell CC 2496944 -> 2320811; Manufacturer (none) -> MULTICOMP; Part number (none) -> MC0603X475K6R3CT
- C7: Descr (none) -> Capacitor X7R 330nF 50V 10% 0603; Farnell CC 1828951 -> 2627440; Manufacturer (none) -> MULTICOMP; Part number (none) -> MC0603B334K250CT
- D1: symbol LED-RESCUE-Doppelganger -> LED; Descr (none) -> Green LED 0805; Manufacturer (none) -> DIALIGHT; Part number (none) -> 5988170107F
- F1, F2, F3: value Fix -> dnf
- FID1, FID2, FID3, FID4, FID5, FID6: value FIDUCIAL -> dnf
- J1: Descr (none) -> RJ45 jack; Manufacturer (none) -> AMPHENOL ICC; Part number (none) -> RJHSE-5380
- J2: value BROOK_FB -> dnf; Farnell CC 1109732 -> 2289780
- P1, P2: Descr (none) -> 10 pin 5mm screw terminal block; Farnell CC (none) -> 9632727; Manufacturer (none) -> IMO PRECISION CONTROLS; Part number (none) -> 20.101M/10
- P3, P4: Descr (none) -> 6 pins 2.54mm connector; Manufacturer (none) -> MULTICOMP; Part number (none) -> 2211S-06G
- P5: Descr (none) -> 3 pins 2.54mm Header single row right angle; Manufacturer (none) -> MULTICOMP; Part number (none) -> MC34747
- P6: Descr (none) -> 4 pin 5mm screw terminal block; Farnell CC (none) -> 9632697; Manufacturer (none) -> IMO PRECISION CONTROLS; Part number (none) -> 20.101M/4
- R1, R25, R26: Descr (none) -> Resistor 330R 100mW 1% 0603; Farnell CC 2502716 -> 2447339; Manufacturer (none) -> MULTICOMP; Part number (none) -> MCWR06X3300FTL
- R10, R11, R12, R13, R14, R15, R16, R17, R18, R19, R2, R20, R22, R23, R24, R28, R3, R4, R5, R6, R7, R8, R9: Descr (none) -> Resistor 10K 100mW 1% 0603; Farnell CC 2447553 -> 2447230; Manufacturer (none) -> MULTICOMP; Part number (none) -> MCWR06X1002FTL
- R21: Descr (none) -> Resistor 100R 100mW 5% 0603; Farnell CC 9333703 -> 2447227; Manufacturer (none) -> MULTICOMP; Part number (none) -> MCWR06X1000FTL
- R27, R29: Descr (none) -> Resistor 3K5 100mW 1% 0603; Farnell CC 2447553 -> 2447361; Manufacturer (none) -> MULTICOMP; Part number (none) -> MCWR06X3481FTL
- R30: Descr (none) -> Resistor 4K7 100mW 1% 0603; Farnell CC 2447553 -> 2694880; Manufacturer (none) -> MULTICOMP; Part number (none) -> MCWR06X472 JTL
- SW1, SW2: value SW_PUSH -> dnf; Farnell CC (none) -> N/A; Manufacturer (none) -> N/A; Part number (none) -> N/A
- U1: Descr (none) -> 4 input OR2 gates; Farnell CC (none) -> 9591427; Manufacturer (none) -> TEXAS INSTRUMENTS; Part number (none) -> SN74HC32D
- U2: Descr (none) -> 44 mOhm load switch; Farnell CC (none) -> 2361514; Manufacturer (none) -> VISHAY; Part number (none) -> SIP32510DT-T1-GE3
- U4, U5, U6: symbol 74LVC07-RESCUE-Doppelganger -> 74LVC07; Descr (none) -> Non inverting hex buffer; Farnell CC (none) -> 9592660; Manufacturer (none) -> TEXAS INSTRUMENTS; Part number (none) -> SN74LVC07ADR
- U4, U5, U6: Descr (none) -> Non inverting hex buffer; Farnell CC (none) -> 9592660; Manufacturer (none) -> TEXAS INSTRUMENTS; Part number (none) -> SN74LVC07ADR
- U8: Descr (none) -> 8 Bit USB Microcontroller; Manufacturer (none) -> MICROCHIP; Part number (none) -> PIC18F45K50-I/PT
- U9: Descr (none) -> 4.5R Quad SPST Analog Switches; Manufacturer (none) -> MAXIM; Part number (none) -> MAX4737EUD+
Connections:
- net GND: now also J3.2 (G2)
- net at J2.J5_6 (ADC_Ry): now also J3.1 (G1)
- no-connect marks 14 -> 8
Other:
- note added: "Fixes"
- note added: "Short to activate\nnew SOCD style:\n<- + -> == -> \n-> + <- == <-"
- moved on the sheet: F1, F2, F3
