File: main_board/Doppelganger.kicad_pcb (KiCad board)
At the start: 2 copper layers, 76.1 x 51.9 mm, 69 parts, among them J1 RJ45, J2 BROOK_FB, P1 BORNIER_10, P2 BORNIER_10, P3 CONN_01X06, P4 CONN_01X06, P5 TTL Serial, P6 Status Leds, SW1 SW_PUSH, SW2 SW_PUSH, U1 74HC32, U2 SIP32510, U4 74LVC07, U5 74LVC07, U6 74LVC07, U8 18F45K50, U9 MAX4737

Commit message: Pre teardrops
Parts:
- removed G***: LOGO, Doppelganger:Sakura_solder_mask
- added J3: dnf, Doppelganger:GS2, F.Cu at (131.2, 112.1)
- added S1: dnf, Doppelganger:Sakura_solder_mask, B.Cu at (128.2, 103.6)
- F1, F2, F3: value Fix -> dnf
- FID1, FID2, FID3, FID4, FID5, FID6: value FIDUCIAL -> dnf
- J2: value BROOK_FB -> dnf
- moved R18 0.86 mm to (119.4, 69.3)
- moved R10 0.86 mm to (139.4, 69.3)
- moved R12 0.86 mm to (134.4, 69.3)
- moved R14 0.86 mm to (129.4, 69.3)
- moved R16 0.86 mm to (124.5, 69.3)
- moved R2 0.86 mm to (159.4, 69.3)
- moved R4 0.86 mm to (154.4, 69.3)
- moved R6 0.86 mm to (149.4, 69.3)
- moved R15 0.81 mm to (103.3, 81.2)
- moved R11 0.81 mm to (103.3, 91.2)
- moved R17 0.81 mm to (103.3, 76.1)
- moved R5 0.81 mm to (103.3, 106.1)
- moved R7 0.81 mm to (103.3, 101.1)
- moved R9 0.81 mm to (103.3, 96.1)
- moved R8 0.46 mm to (142.8, 73.8)
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Connections:
- J2 pad J5_6: (no net) -> Net-(J2-PadJ5_6)
Routing:
- net (no net): track 211.0 -> 0.00 mm
- net /CSS1: track 61.4 -> 54.9 mm, vias 5 -> 4
- net /B_PS_KEY: track 14.3 -> 20.6 mm
- net /UP: track 118.7 -> 112.9 mm
- net GND: track 83.3 -> 88.0 mm
- net /B_START: track 33.9 -> 38.5 mm
- net /Disable: track 101.2 -> 97.0 mm
- net /USB_INPUT-: track 73.6 -> 69.6 mm, vias 7 -> 5
- net /PS_KEY: track 70.5 -> 66.7 mm
- net /START: track 76.7 -> 73.1 mm
- net /L3: track 85.8 -> 82.3 mm
- net /DOWN: track 95.4 -> 92.0 mm
- net /Uart_Tx: track 46.7 -> 49.9 mm
- net /B_SELECT: track 49.8 -> 46.6 mm
- net /R1: track 59.2 -> 56.1 mm
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Other:
- net class Default: clearance 0.1524 -> 0.2032; trace_width 0.1524 -> 0.2032
- net class USB: clearance 0.254 -> 0.2032; trace_width 0.254 -> 0.2032; via_dia 0.6 -> 0.508
- rule trace_clearance: 0.1524 -> 0.2032
- rule via_min_drill: 0.3 -> 0.254
- rule via_min_size: 0.4 -> 0.254
- board text added: "Short J3 to activate Brook new SOCD mode"

Commit message: RevB0
Other:
- net class Leds: clearance 0.254 -> 0.2032
- rule trace_min: 0.1524 -> 0.2032
