File: usb_alien/_autosave-usb_alien.kicad_pcb (KiCad board)
At the start: 2 copper layers, 40.6 x 40.7 mm, 15 parts, among them J1 BROOK_FB, J2 HE10-12X2, J3 GS2, J4 GS2, J5 GS2, P1 BORNIER_4, P2 BORNIER_4, P3 BORNIER_10, P4 BORNIER_10, U1 74HC00, U2 74HC00

Commit message: RevB0
Parts:
- C2: value C -> 100nF
Changed lines of the file:
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@@
-(kicad_pcb (version 20170922) (host pcbnew no-vcs-found-1164eaa~60~ubuntu16.04.1)
+(kicad_pcb (version 20170922) (host pcbnew no-vcs-found-f685cfa~60~ubuntu16.04.1)
 (general
   (thickness 1.6)
-  (drawings 12)
+  (drawings 14)
   (tracks 494)
   (zones 0)
@@
 (page A4)
 (layers
-  (0 F.Cu signal)
-  (31 B.Cu signal)
-  (32 B.Adhes user)
-  (33 F.Adhes user)
+  (0 F.Cu signal hide)
+  (31 B.Cu signal hide)
+  (32 B.Adhes user hide)
+  (33 F.Adhes user hide)
   (34 B.Paste user)
   (35 F.Paste user)
   (36 B.SilkS user)
   (37 F.SilkS user)
-  (38 B.Mask user)
-  (39 F.Mask user)
+  (38 B.Mask user hide)
+  (39 F.Mask user hide)
   (40 Dwgs.User user)
   (41 Cmts.User user)
@@
 (general
   (thickness 1.6)
-  (drawings 12)
+  (drawings 14)
   (tracks 494)
   (zones 0)
@@
 (page A4)
 (layers
-  (0 F.Cu signal)
-  (31 B.Cu signal)
-  (32 B.Adhes user)
-  (33 F.Adhes user)
+  (0 F.Cu signal hide)
+  (31 B.Cu signal hide)
+  (32 B.Adhes user hide)
+  (33 F.Adhes user hide)
   (34 B.Paste user)
   (35 F.Paste user)
   (36 B.SilkS user)
   (37 F.SilkS user)
-  (38 B.Mask user)
-  (39 F.Mask user)
+  (38 B.Mask user hide)
+  (39 F.Mask user hide)
   (40 Dwgs.User user)
   (41 Cmts.User user)
@@
   (pad_to_mask_clearance 0.2)
   (aux_axis_origin 0 0)
-  (visible_elements FFFDFF7F)
+  (visible_elements FFFDFF77)
   (pcbplotparams
-    (layerselection 0x00030_ffffffff)
-    (usegerberextensions false)
+    (layerselection 0x010f0_ffffffff)
+    (usegerberextensions true)
     (usegerberattributes true)
     (usegerberadvancedattributes true)
@@
     (outputformat 1)
     (mirror false)
-    (drillshape 1)
+    (drillshape 0)
     (scaleselection 1)
-    (outputdirectory ""))
+    (outputdirectory fabrication/RevB0/Drill/))
 )
 (net 0 "")
@@
       (effects (font (size 1 1) (thickness 0.15)))
     )
-    (fp_text value C (at 0.635 1.905 90) (layer F.Fab)
+    (fp_text value 100nF (at 0.635 1.905 90) (layer F.Fab)
       (effects (font (size 1 1) (thickness 0.15)))
     )
@@
     )
   )
+  (dimension 40.65 (width 0.3) (layer F.Fab)
+    (gr_text "40,650 mm" (at 143.575 113.9) (layer F.Fab)
+      (effects (font (size 1.5 1.5) (thickness 0.3)))
+    )
+    (feature1 (pts (xy 163.9 110.65) (xy 163.9 115.25)))
+    (feature2 (pts (xy 123.25 110.65) (xy 123.25 115.25)))
+    (crossbar (pts (xy 123.25 112.55) (xy 163.9 112.55)))
+    (arrow1a (pts (xy 163.9 112.55) (xy 162.773496 113.136421)))
+    (arrow1b (pts (xy 163.9 112.55) (xy 162.773496 111.963579)))
+    (arrow2a (pts (xy 123.25 112.55) (xy 124.376504 113.136421)))
+    (arrow2b (pts (xy 123.25 112.55) (xy 124.376504 111.963579)))
+  )
+  (dimension 40.65 (width 0.3) (layer F.Fab)
+    (gr_text "40,650 mm" (at 170.65 90.325 270) (layer F.Fab)
+      (effects (font (size 1.5 1.5) (thickness 0.3)))
+    )
+    (feature1 (pts (xy 163.9 110.65) (xy 172 110.65)))
+    (feature2 (pts (xy 163.9 70) (xy 172 70)))
+    (crossbar (pts (xy 169.3 70) (xy 169.3 110.65)))
+    (arrow1a (pts (xy 169.3 110.65) (xy 168.713579 109.523496)))
+    (arrow1b (pts (xy 169.3 110.65) (xy 169.886421 109.523496)))
+    (arrow2a (pts (xy 169.3 70) (xy 168.713579 71.126504)))
+    (arrow2b (pts (xy 169.3 70) (xy 169.886421 71.126504)))
+  )
   (gr_text "Rev B0" (at 131.8641 75.2856) (layer B.SilkS)
