File: usb_alien/usb_alien.kicad_pcb (KiCad board)
At the start: 2 copper layers, 40.6 x 40.7 mm, 15 parts, among them J1 BROOK_FB, J2 HE10-12X2, J3 GS2, J4 GS2, J5 GS2, P1 BORNIER_4, P2 BORNIER_4, P3 BORNIER_10, P4 BORNIER_10, U1 74HC00, U2 74HC00

Commit message: RevB0
Parts:
- C2: value C -> 100nF
