File: arcade_adapter/arcade_adapter.kicad_pcb (KiCad board)
At the start: 2 copper layers, 22 x 39 mm, 14 parts, among them J1 RJ45, J2 CONN_01X06, J3 DB15_FEMALE, U1 18F23K22

Commit message: Arcade adapter RevB1 first commit
Parts:
- removed G***: LOGO, Doppelganger:CAMMIE_SOLDER_MASK
- J3: moved to B.Cu
- moved J3 19.5 mm to (111.3, 57.3), turned to 180 degrees
- moved R3 5.86 mm to (106.8, 65.7), turned to 180 degrees
- moved C1 4.40 mm to (106.8, 67.6)
Connections:
- J1 pad 3: /SDI -> /MISO
- J1 pad 4: /SDO -> /MOSI
- J3 pad 1: VDD -> GND
- J3 pad 10: /Left -> /MK
- J3 pad 11: /LP -> /Start
- J3 pad 13: /Start -> /LP
- J3 pad 14: /MK -> /Left
- J3 pad 15: Net-(J3-Pad15) -> /Up
- J3 pad 2: /Down -> /HK
- J3 pad 3: /Right -> /Coin
- J3 pad 4: /MP -> /LK
- J3 pad 5: /LK -> /MP
- J3 pad 6: /Coin -> /Right
- J3 pad 7: /HK -> /Down
- J3 pad 8: GND -> VDD
- J3 pad 9: /Up -> /NC
- U1 pad 15: /SDI -> /MOSI
- U1 pad 16: /SDO -> /MISO
- U1 pad 25: Net-(U1-Pad25) -> /NC
Routing:
- net /SDI: track 28.2 -> 0.00 mm, vias 3 -> 0
- net /MISO: track 0.00 -> 27.4 mm, vias 0 -> 3
- net /MOSI: track 0.00 -> 25.4 mm, vias 0 -> 3
- net /SDO: track 24.8 -> 0.00 mm, vias 3 -> 0
- net /NC: track 0.00 -> 21.5 mm, vias 0 -> 2
- net Net-(C1-Pad1): track 29.9 -> 23.4 mm
- net GND: track 29.2 -> 33.5 mm, vias 14 -> 20
- net /Up: track 9.57 -> 5.90 mm, vias 1 -> 0
- net VDD: track 20.9 -> 18.7 mm
- net /SCK: track 38.0 -> 36.5 mm
- net /Coin: track 5.97 -> 5.72 mm, vias 0 -> 1
- net /HK: track 6.08 -> 5.83 mm, vias 0 -> 1
- net /MP: track 16.6 -> 16.8 mm, vias 2 -> 1
- net /LP: track 5.93 -> 5.69 mm, vias 1 -> 0
- net /HP: track 16.0 -> 16.2 mm, vias 1 -> 2
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- removed copper zone on B.Cu, net (none)
Other:
- outline, holes or cut-outs redrawn
- board text added: "Doppelganger Arcade Adapter Rev B1"
- board text added: "© 2018 Niluje"
- board text removed: "Doppelganger Arcade Adapter Rev B0"
- board text removed: "© 2017 Niluje"
