File: arcade_adapter/arcade_adapter.sch (KiCad schematic (older format))
At the start: 13 parts, among them J1 RJ45, J2 CONN_01X06, J3 DB15_FEMALE, U1 18F23K22

Commit message: Arcade adapter RevB1 first commit
Parts:
- C1, C2, C3: symbol C -> arcade_adapter-rescue:C-RESCUE-arcade_adapter
- D1, D2: symbol LED -> arcade_adapter-rescue:LED-RESCUE-arcade_adapter
- J1: symbol RJ45 -> arcade_adapter-rescue:RJ45-RESCUE-arcade_adapter
- J2: symbol CONN_01X06 -> arcade_adapter-rescue:CONN_01X06-RESCUE-arcade_adapter
- J3: symbol DB15_FEMALE -> arcade_adapter-rescue:DB15_FEMALE-RESCUE-arcade_adapter
- R1, R2, R3, R4: symbol R -> arcade_adapter-rescue:R-RESCUE-arcade_adapter
- U1: symbol 18F23K22 -> arcade_adapter-rescue:18F23K22-RESCUE-arcade_adapter
Connections:
- net Coin: now also J3.3; no longer J3.6
- net Down: now also J3.7; no longer J3.2
- net GND: now also J3.1; no longer J3.8
- net HK: now also J3.2; no longer J3.7
- net LK: now also J3.4; no longer J3.5
- net LP: now also J3.13 (P13); no longer J3.11 (P111)
- net Left: now also J3.14 (P14); no longer J3.10 (P10)
- net MK: now also J3.10 (P10); no longer J3.14 (P14)
- net MP: now also J3.5; no longer J3.4
- net Right: now also J3.6; no longer J3.3
- net Start: now also J3.11 (P111); no longer J3.13 (P13)
- net Up: now also J3.15 (P15); no longer J3.9 (P9)
- net VDD: now also J3.8; no longer J3.1
- net NC: now reaches U1.25 (RB4)
- net NC: now also J3.9 (P9)
- net SDI renamed MISO
- net MISO: now also U1.16 (SD0); no longer U1.15 (SDI)
- net SDO renamed MOSI
- net MOSI: now also U1.15 (SDI); no longer U1.16 (SD0)
- no-connect marks 5 -> 3
Other:
- note added: "Button attribution is done according to the UD USB decoder.\n(See http://udgametech.blogspot.fr/p/products.html).\nNC remains connected in order to handle multiple mapping (smallcab, MAK Strike)."
- moved on the sheet: J3
